Commit message: feat(description): carry the AGX gripper in the Duo model and its gravity
The Duo body description knew only the OmniHand, so an arm wearing the AGX
gripper was modelled bare. The gravity URDF ended at nero_tool0 with a 1e-6 kg
placeholder while 0.548 kg hung on the flange, uncompensated at the longest
lever arm of the chain.

- Each side can now take either the hand or the gripper on the shared link7
  tool mount; the gravity slice folds in whichever is mounted, raising the right
  arm's modelled mass from 4.580 to 5.128 kg.
- The gripper's two prismatic fingers are frozen in the gravity URDF: 0.025 kg
  each against 0.498 kg of flange and base, so their pose does not move the
  arm's gravity torque and the model needs no finger feedback.
- Gripper commands now go through the arm's SDK worker on the control lane
  instead of reaching the vendor SDK from a subscription callback. The gripper
  shares the arm's session and CAN socket, so it was the one remaining writer
  outside the single-owner rule. A superseded target is dropped while queued.
- Inertials are the SolidWorks values already carried by the single-arm gripper
  description, not estimates.

Validation: package tests and generated-URDF inspection. Not exercised on
hardware: whether the corrected gravity model holds the arm steady is unproven,
and the arm's idle-hold behaviour with this gripper mounted is an open question.

File: src/duo_body_description/urdf/duo_system.urdf.xacro (robot description, xacro)
@@ -5,4 +5,8 @@
   <xacro:arg name="use_right_arm" default="true"/>
   <xacro:arg name="use_right_hand" default="true"/>
+  <!-- A side takes either the hand or the gripper: both mount on the same
+       link7 frame. The launch layer refuses the pair; xacro cannot raise. -->
+  <xacro:arg name="use_left_gripper" default="false"/>
+  <xacro:arg name="use_right_gripper" default="false"/>
   <xacro:arg name="left_arm_prefix" default="left_arm_"/>
   <xacro:arg name="right_arm_prefix" default="right_arm_"/>
@@ -34,4 +38,8 @@
       <xacro:omnihand_hand arm_prefix="${left_arm_prefix}" hand_side="left"/>
     </xacro:if>
+    <xacro:if value="$(arg use_left_gripper)">
+      <xacro:agx_gripper_flange arm_prefix="${left_arm_prefix}"/>
+      <xacro:agx_gripper arm_prefix="${left_arm_prefix}"/>
+    </xacro:if>
   </xacro:if>
   <xacro:if value="$(arg use_right_arm)">
@@ -46,4 +54,8 @@
       <xacro:omnihand_hand arm_prefix="${right_arm_prefix}" hand_side="right"/>
     </xacro:if>
+    <xacro:if value="$(arg use_right_gripper)">
+      <xacro:agx_gripper_flange arm_prefix="${right_arm_prefix}"/>
+      <xacro:agx_gripper arm_prefix="${right_arm_prefix}"/>
+    </xacro:if>
   </xacro:if>
 </robot>

File: src/duo_body_description/urdf/nero_arm_macro.xacro (robot description, xacro)
@@ -290,3 +290,114 @@
     </xacro:if>
   </xacro:macro>
+  <!-- AGX gripper, side-prefixed. Same link7 tool mount as omnihand_flange, so
+       the two are alternatives on one arm, never both. Inertials are the
+       SolidWorks values from agx_arm_description's single-arm gripper xacro;
+       the gravity model needs them at 0.548 kg total. -->
+  <xacro:macro name="agx_gripper_flange" params="arm_prefix">
+    <link name="${arm_prefix}gripper_flange">
+      <inertial>
+        <origin xyz="0.0 0.0 -0.00032" rpy="0 0 0"/>
+        <mass value="0.04771096"/>
+        <inertia ixx="2.697e-05" ixy="0" ixz="0" iyy="4.311e-05" iyz="0" izz="2.479e-05"/>
+      </inertial>
+      <visual>
+        <origin xyz="0 0 0" rpy="0 0 0"/>
+        <geometry>
+          <mesh filename="package://agx_arm_description/agx_arm_urdf/nero/meshes/dae/gripper_flange.dae"/>
+        </geometry>
+      </visual>
+      <collision>
+        <origin xyz="0 0 0" rpy="0 0 0"/>
+        <geometry>
+          <mesh filename="package://agx_arm_description/agx_arm_urdf/nero/meshes/gripper_flange.stl"/>
+        </geometry>
+      </collision>
+    </link>
+    <joint name="${arm_prefix}gripper_flange_joint" type="fixed">
+      <origin xyz="0.032 0 -0.0235" rpy="-1.5708 0 -1.5708"/>
+      <parent link="${arm_prefix}link7"/>
+      <child link="${arm_prefix}gripper_flange"/>
+    </joint>
+  </xacro:macro>
+  <!-- The two finger joints are prismatic and mirror each other; the driver
+       publishes them as gripper_joint1/2 at +/-0.5 * measured width, which the
+       joint_state_merger then prefixes. -->
+  <xacro:macro name="agx_gripper" params="arm_prefix">
+    <link name="${arm_prefix}gripper_base">
+      <inertial>
+        <origin xyz="-0.000183807162235591 8.05033155577911E-05 0.0321436689908876" rpy="0 0 0"/>
+        <mass value="0.45"/>
+        <inertia ixx="0.00092934" ixy="0.00000034" ixz="-0.00000738" iyy="0.00071447" iyz="0.00000005" izz="0.00039442"/>
+      </inertial>
+      <visual>
+        <origin xyz="0 0 0" rpy="0 0 0"/>
+        <geometry>
+          <mesh filename="package://agx_arm_description/agx_arm_urdf/nero/meshes/dae/gripper_base.dae"/>
+        </geometry>
+      </visual>
+      <collision>
+        <origin xyz="0 0 0" rpy="0 0 0"/>
+        <geometry>
+          <mesh filename="package://agx_arm_description/agx_arm_urdf/nero/meshes/gripper_base.stl"/>
+        </geometry>
+      </collision>
+    </link>
+    <joint name="${arm_prefix}gripper_base_joint" type="fixed">
+      <origin xyz="0 0 0.0055" rpy="0 0 0"/>
+      <parent link="${arm_prefix}gripper_flange"/>
+      <child link="${arm_prefix}gripper_base"/>
+    </joint>
+    <link name="${arm_prefix}gripper_link1">
+      <inertial>
+        <origin xyz="0.00065123185041968 -0.0491929869131989 0.00972258769184025" rpy="0 0 0"/>
+        <mass value="0.025"/>
+        <inertia ixx="0.00007371" ixy="-0.00000113" ixz="0.00000021" iyy="0.00000781" iyz="-0.00001372" izz="0.0000747"/>
+      </inertial>
+      <visual>
+        <origin xyz="0 0 0" rpy="0 0 0"/>
+        <geometry>
+          <mesh filename="package://agx_arm_description/agx_arm_urdf/nero/meshes/dae/gripper_link1.dae"/>
+        </geometry>
+      </visual>
+      <collision>
+        <origin xyz="0 0 0" rpy="0 0 0"/>
+        <geometry>
+          <mesh filename="package://agx_arm_description/agx_arm_urdf/nero/meshes/gripper_link1.stl"/>
+        </geometry>
+      </collision>
+    </link>
+    <joint name="${arm_prefix}gripper_joint1" type="prismatic">
+      <origin xyz="0 0 0.1358" rpy="1.5707963 0 3.1415926"/>
+      <parent link="${arm_prefix}gripper_base"/>
+      <child link="${arm_prefix}gripper_link1"/>
+      <axis xyz="0 0 1"/>
+      <limit lower="0" upper="0.05" effort="10" velocity="3"/>
+    </joint>
+    <link name="${arm_prefix}gripper_link2">
+      <inertial>
+        <origin xyz="0.00065123185041968 -0.0491929869131989 0.00972258769184025" rpy="0 0 0"/>
+        <mass value="0.025"/>
+        <inertia ixx="0.00007371" ixy="-0.00000113" ixz="0.00000021" iyy="0.00000781" iyz="-0.00001372" izz="0.0000747"/>
+      </inertial>
+      <visual>
+        <origin xyz="0 0 0" rpy="0 0 0"/>
+        <geometry>
+          <mesh filename="package://agx_arm_description/agx_arm_urdf/nero/meshes/dae/gripper_link2.dae"/>
+        </geometry>
+      </visual>
+      <collision>
+        <origin xyz="0 0 0" rpy="0 0 0"/>
+        <geometry>
+          <mesh filename="package://agx_arm_description/agx_arm_urdf/nero/meshes/gripper_link2.stl"/>
+        </geometry>
+      </collision>
+    </link>
+    <joint name="${arm_prefix}gripper_joint2" type="prismatic">
+      <origin xyz="0 0 0.1358" rpy="1.5707963 0 0"/>
+      <parent link="${arm_prefix}gripper_base"/>
+      <child link="${arm_prefix}gripper_link2"/>
+      <axis xyz="0 0 -1"/>
+      <limit lower="-0.05" upper="0" effort="10" velocity="3"/>
+    </joint>
+  </xacro:macro>
 </robot>
