Commit message: Feat: Prepare common body two arm config and sprint targets.

File: src/duo_body_description/urdf/duo_body.xacro (robot description, xacro)
@@ -1,16 +1,17 @@
 <?xml version="1.0"?>
 <robot xmlns:xacro="http://www.ros.org/wiki/xacro">
-  <xacro:macro name="duo_body">
+  <!--<xacro:macro name="duo_body" params="body_mesh_xyz:='-0.11 -0.12411761856079102 -0.07' body_mesh_rpy:='0 0 0'">-->
+  <xacro:macro name="duo_body" params="body_mesh_xyz:='0 0 0' body_mesh_rpy:='0 0 0'">
     <link name="body_base_link">
       <visual>
-        <origin xyz="0 0 0" rpy="0 0 0"/>
+        <origin xyz="${body_mesh_xyz}" rpy="${body_mesh_rpy}"/>
         <geometry>
-          <mesh filename="package://duo_body_description/meshes/body_visual.stl"/>
+          <mesh filename="package://duo_body_description/meshes/body_visual.stl" scale="0.001 0.001 0.001"/>
         </geometry>
       </visual>
       <collision>
-        <origin xyz="0 0 0" rpy="0 0 0"/>
+        <origin xyz="${body_mesh_xyz}" rpy="${body_mesh_rpy}"/>
         <geometry>
-          <mesh filename="package://duo_body_description/meshes/body_collision.stl"/>
+          <mesh filename="package://duo_body_description/meshes/body_collision.stl" scale="0.001 0.001 0.001"/>
         </geometry>
       </collision>
@@ -20,5 +21,5 @@
       <parent link="body_base_link"/>
       <child link="left_arm_mount_link"/>
-      <origin xyz="-0.136240 0.105467 0.070150" rpy="0 1.570796 -0.837758"/>
+      <origin xyz="-0.137511 0.104055 0.070000" rpy="0 1.570796 -0.837758"/>
     </joint>
     <link name="right_arm_mount_link"/>

File: src/duo_body_description/urdf/duo_system.urdf.xacro (robot description, xacro)
@@ -7,7 +7,12 @@
   <xacro:arg name="left_arm_prefix" default="left_arm_"/>
   <xacro:arg name="right_arm_prefix" default="right_arm_"/>
-  <xacro:arg name="left_arm_base_xyz" default="0 0 0"/>
-  <xacro:arg name="left_arm_base_rpy" default="0 0 0"/>
-  <xacro:arg name="right_arm_base_xyz" default="0 0 0"/>
+  <!--<xacro:arg name="body_mesh_xyz" default="-0.11 -0.12411761856079102 -0.07"/>-->
+  <xacro:arg name="body_mesh_xyz" default="0 0 0"/>
+  <xacro:arg name="body_mesh_rpy" default="0 0 0"/>
+  <xacro:arg name="left_arm_base_xyz" default="0.01 0.02 0"/>
+  <xacro:arg name="left_arm_base_rpy" default="0 0 3.1415926"/>
+  <!--<xacro:arg name="right_arm_base_xyz" default="-0.01 -0.02 0"/>-->
+  <xacro:arg name="right_arm_base_xyz" default="0.0 0.0 0.0"/>
+  <!--<xacro:arg name="right_arm_base_rpy" default="0 0 3.1415926"/>-->
   <xacro:arg name="right_arm_base_rpy" default="0 0 0"/>
   <xacro:property name="left_arm_prefix" value="$(arg left_arm_prefix)"/>
@@ -15,5 +20,5 @@
   <xacro:include filename="$(find duo_body_description)/urdf/duo_body.xacro"/>
   <xacro:include filename="$(find duo_body_description)/urdf/nero_arm_macro.xacro"/>
-  <xacro:duo_body/>
+  <xacro:duo_body body_mesh_xyz="$(arg body_mesh_xyz)" body_mesh_rpy="$(arg body_mesh_rpy)"/>
   <xacro:if value="$(arg use_left_arm)">
     <xacro:nero_arm prefix="${left_arm_prefix}"/>

Commit message: fix(duo-bringup): enable per-arm drivers and CAN ports in duo_arm profile
- execution_profiles.yaml: duo_arm arm instances now have launch_driver:true
  and explicit can_port (can_nero_left / can_nero_right)
- start_multi_agx_arm_rviz.launch.py: declare arm_base_frame/arm_tip_frame args
- start_moveit.launch.py: body_base_link as RViz fixed frame for custom models (staged)
- duo_body.xacro: fix left arm mount pitch sign (0 1.57 → 0 -1.57)
- duo_system.urdf.xacro: fix left_arm_base_rpy yaw sign (+π/2 → -π/2)

File: src/duo_body_description/urdf/duo_body.xacro (robot description, xacro)
@@ -22,5 +22,5 @@
       <child link="left_arm_mount_link"/>
       <!--<origin xyz="-0.137511 0.104055 0.070000" rpy="0 1.570796 -0.837758"/>-->
-      <origin xyz="-0.154602 0.110059 0.078262" rpy="0 1.570796 -0.837758"/>
+      <origin xyz="-0.154602 0.110059 0.078262" rpy="0 -1.570796 -0.837758"/>
     </joint>
     <link name="right_arm_mount_link"/>

File: src/duo_body_description/urdf/duo_system.urdf.xacro (robot description, xacro)
@@ -13,5 +13,5 @@
   <xacro:arg name="left_arm_base_xyz" default="0.0 0.0 0.0"/>
   <!--<xacro:arg name="left_arm_base_rpy" default="0 0 3.1415926"/>-->
-  <xacro:arg name="left_arm_base_rpy" default="0 0 1.570796"/>
+  <xacro:arg name="left_arm_base_rpy" default="0 0 -1.570796"/>
   <!--<xacro:arg name="right_arm_base_xyz" default="-0.01 -0.02 0"/>-->
   <xacro:arg name="right_arm_base_xyz" default="0.0 0.0 0.0"/>
