Commit message: chore(nero): align active docs and launches to nero

File: src/agx_arm_moveit/config/agx_arm.srdf.xacro (robot description, xacro)
@@ -1,9 +1,9 @@
 <?xml version="1.0" encoding="UTF-8"?>
 <robot xmlns:xacro="http://www.ros.org/wiki/xacro" name="agx_arm">
-  <xacro:arg name="arm_type" default="piper" />
+  <xacro:arg name="arm_type" default="nero" />
   <xacro:arg name="effector_type" default="none" />
   <xacro:arg name="revo2_type" default="left" />
   <xacro:property name="arm_type" value="$(arg arm_type)" />
-  <xacro:property name="flange_link" value="${'link7' if arm_type == 'nero' else 'link6'}" />
+  <xacro:property name="flange_link" value="link7" />
   <!-- ======================== ARM GROUP ======================== -->
   <group name="arm">

File: src/agx_arm_moveit/config/agx_arm.urdf.xacro (robot description, xacro)
@@ -1,5 +1,5 @@
 <?xml version="1.0"?>
 <robot xmlns:xacro="http://www.ros.org/wiki/xacro" name="agx_arm">
-  <xacro:arg name="arm_type" default="piper" />
+  <xacro:arg name="arm_type" default="nero" />
   <xacro:arg name="effector_type" default="none" />
   <xacro:arg name="revo2_type" default="left" />
@@ -8,5 +8,5 @@
   <xacro:arg name="tcp_offset_rpy" default="0 0 0" />
   <xacro:property name="arm_type" value="$(arg arm_type)" />
-  <xacro:property name="flange_link" value="${'link7' if arm_type == 'nero' else 'link6'}" />
+  <xacro:property name="flange_link" value="link7" />
   <xacro:if value="$(eval effector_type == 'agx_gripper')">
     <xacro:include filename="$(find agx_arm_description)/agx_arm_urdf/$(arg arm_type)/urdf/$(arg arm_type)_with_gripper_description.xacro" />

Commit message: feat(sprint3): harden nero MoveIt baseline and docs
Align the active Nero MoveIt surface on the nero_arm planning group, the nero_tool0 flange alias, and a TRAC-IK kinematics baseline.

Add Sprint 3 working notes plus a multi-profile MoveIt smoke helper, document the conditional TRAC-IK install/source flow, and record the remaining Humble/aarch64 move_group shutdown gate.

Follow up on review findings by avoiding Nero-specific tcp_link injection for custom RViz models and by restoring the legacy nero_gripper_moveit_config kinematics key to match its renamed SRDF group.

File: src/agx_arm_moveit/config/agx_arm.srdf.xacro (robot description, xacro)
@@ -20,5 +20,5 @@
       <joint name="${side}_pinky_pip_joint" />
     </group>
-    <end_effector name="${side}_omnihand_eef" parent_link="tcp_link" group="hand" parent_group="arm" />
+    <end_effector name="${side}_omnihand_eef" parent_link="tcp_link" group="hand" parent_group="nero_arm" />
     <group_state name="hand_open" group="hand">
       <joint name="${side}_thumb_roll_joint" value="0.0" />
@@ -86,6 +86,6 @@
     <disable_collisions link1="${side}_pinky_pip" link2="${side}_pinky_dip" reason="Adjacent" />
   </xacro:macro>
-  <!-- ======================== ARM GROUP ======================== -->
-  <group name="arm">
+  <!-- ======================== ARM GROUPS ======================== -->
+  <group name="nero_arm">
     <chain base_link="base_link" tip_link="tcp_link" />
   </group>
@@ -99,5 +99,5 @@
       <joint name="gripper_joint2" />
     </group>
-    <end_effector name="gripper_eef" parent_link="tcp_link" group="gripper" parent_group="arm" />
+    <end_effector name="gripper_eef" parent_link="tcp_link" group="gripper" parent_group="nero_arm" />
     <group_state name="gripper_open" group="gripper">
       <joint name="gripper_joint1" value="0.05" />
@@ -150,5 +150,5 @@
       <link name="left_pinky_distal_link" />
     </group>
-    <end_effector name="left_hand_eef" parent_link="tcp_link" group="hand" parent_group="arm" />
+    <end_effector name="left_hand_eef" parent_link="tcp_link" group="hand" parent_group="nero_arm" />
     <group_state name="hand_open" group="hand">
       <joint name="left_thumb_metacarpal_joint" value="0.0" />
@@ -295,5 +295,5 @@
       <link name="right_pinky_distal_link" />
     </group>
-    <end_effector name="right_hand_eef" parent_link="tcp_link" group="hand" parent_group="arm" />
+    <end_effector name="right_hand_eef" parent_link="tcp_link" group="hand" parent_group="nero_arm" />
     <group_state name="hand_open" group="hand">
       <joint name="right_thumb_metacarpal_joint" value="0.0" />
@@ -426,16 +426,6 @@
   </xacro:if>
   <!-- ======================== HOME STATE ======================== -->
-  <xacro:unless value="$(eval arm_type == 'nero')">
-    <group_state name="home" group="arm">
-      <joint name="joint1" value="0" />
-      <joint name="joint2" value="0" />
-      <joint name="joint3" value="0" />
-      <joint name="joint4" value="0" />
-      <joint name="joint5" value="0" />
-      <joint name="joint6" value="0" />
-    </group_state>
-  </xacro:unless>
   <xacro:if value="$(eval arm_type == 'nero')">
-    <group_state name="home" group="arm">
+    <group_state name="home" group="nero_arm">
       <joint name="joint1" value="0" />
       <joint name="joint2" value="0" />
@@ -477,12 +467,4 @@
     <disable_collisions link1="link5" link2="link7" reason="Never" />
     <disable_collisions link1="link6" link2="link7" reason="Adjacent" />
-    <xacro:if value="$(eval effector_type == 'none')">
-      <disable_collisions link1="base_link" link2="end_effector" reason="Never" />
-      <disable_collisions link1="end_effector" link2="link1" reason="Never" />
-      <disable_collisions link1="end_effector" link2="link2" reason="Never" />
-      <disable_collisions link1="end_effector" link2="link3" reason="Never" />
-      <disable_collisions link1="end_effector" link2="link4" reason="Never" />
-      <disable_collisions link1="end_effector" link2="link7" reason="Adjacent" />
-    </xacro:if>
   </xacro:if>
 </robot>

File: src/agx_arm_moveit/config/agx_arm.urdf.xacro (robot description, xacro)
@@ -9,5 +9,5 @@
   <xacro:arg name="tcp_offset_rpy" default="0 0 0" />
   <xacro:property name="arm_type" value="$(arg arm_type)" />
-  <xacro:property name="flange_link" value="link7" />
+  <xacro:property name="flange_link" value="nero_tool0" />
   <xacro:if value="$(eval effector_type == 'agx_gripper')">
     <xacro:include filename="$(find agx_arm_description)/agx_arm_urdf/$(arg arm_type)/urdf/$(arg arm_type)_with_gripper_description.xacro" />
@@ -28,5 +28,5 @@
     <xacro:include filename="$(find agx_arm_description)/agx_arm_urdf/$(arg arm_type)/urdf/$(arg arm_type)_description.urdf" />
   </xacro:if>
-  <!-- TCP link: fixed offset from flange for MoveIt planning target -->
+  <!-- TCP link: fixed offset from the canonical Nero flange alias for MoveIt planning targets. -->
   <link name="tcp_link" />
   <joint name="tcp_joint" type="fixed">

File: src/agx_arm_sim/agx_arm_description/agx_arm_urdf/nero/urdf/nero_description.urdf (robot description, URDF)
Before this commit: robot nero, 9 links, 8 joints
Links:
- added link nero_tool0
Joints:
- added joint nero_tool0_joint: type fixed, parent link7, child nero_tool0, origin xyz=0 0 0 rpy=0 0 0

File: src/agx_arm_sim/agx_arm_description/urdf/nero_gripper_d435.urdf (robot description, URDF)
Before this commit: robot agx_arm, 17 links, 16 joints
Links:
- added link nero_tool0
Joints:
- added joint nero_tool0_joint: type fixed, parent link7, child nero_tool0, origin xyz=0 0 0 rpy=0 0 0
