Commit message: Land Sprint 4 duo hand-aware runtime slice

File: src/agx_arm_moveit/config/agx_arm.srdf.xacro (robot description, xacro)
@@ -9,4 +9,6 @@
   <xacro:arg name="arm_base_frame" default="base_link" />
   <xacro:arg name="arm_tip_frame" default="tcp_link" />
+  <xacro:arg name="end_effector_parent_link" default="tcp_link" />
+  <xacro:arg name="mount_body_link" default="" />
   <xacro:arg name="arm_joint_prefix" default="" />
   <xacro:arg name="arm_link_prefix" default="" />
@@ -15,8 +17,10 @@
   <xacro:arg name="left_arm_base_frame" default="left_arm_base_link" />
   <xacro:arg name="left_arm_tip_frame" default="left_arm_nero_tool0" />
+  <xacro:arg name="left_mount_body_link" default="" />
   <xacro:arg name="left_arm_joint_prefix" default="left_arm_" />
   <xacro:arg name="left_arm_link_prefix" default="left_arm_" />
   <xacro:arg name="right_arm_base_frame" default="right_arm_base_link" />
   <xacro:arg name="right_arm_tip_frame" default="right_arm_nero_tool0" />
+  <xacro:arg name="right_mount_body_link" default="" />
   <xacro:arg name="right_arm_joint_prefix" default="right_arm_" />
   <xacro:arg name="right_arm_link_prefix" default="right_arm_" />
@@ -26,4 +30,6 @@
   <xacro:property name="arm_base_frame" value="$(arg arm_base_frame)" />
   <xacro:property name="arm_tip_frame" value="$(arg arm_tip_frame)" />
+  <xacro:property name="end_effector_parent_link" value="$(arg end_effector_parent_link)" />
+  <xacro:property name="mount_body_link" value="$(arg mount_body_link)" />
   <xacro:property name="arm_joint_prefix" value="$(arg arm_joint_prefix)" />
   <xacro:property name="arm_link_prefix" value="$(arg arm_link_prefix)" />
@@ -31,8 +37,10 @@
   <xacro:property name="left_arm_base_frame" value="$(arg left_arm_base_frame)" />
   <xacro:property name="left_arm_tip_frame" value="$(arg left_arm_tip_frame)" />
+  <xacro:property name="left_mount_body_link" value="$(arg left_mount_body_link)" />
   <xacro:property name="left_arm_joint_prefix" value="$(arg left_arm_joint_prefix)" />
   <xacro:property name="left_arm_link_prefix" value="$(arg left_arm_link_prefix)" />
   <xacro:property name="right_arm_base_frame" value="$(arg right_arm_base_frame)" />
   <xacro:property name="right_arm_tip_frame" value="$(arg right_arm_tip_frame)" />
+  <xacro:property name="right_mount_body_link" value="$(arg right_mount_body_link)" />
   <xacro:property name="right_arm_joint_prefix" value="$(arg right_arm_joint_prefix)" />
   <xacro:property name="right_arm_link_prefix" value="$(arg right_arm_link_prefix)" />
@@ -53,34 +61,14 @@
     </group_state>
   </xacro:macro>
-  <xacro:macro name="nero_arm_disable_collisions" params="link_prefix">
+  <xacro:macro name="nero_arm_disable_collisions" params="link_prefix mount_body_link">
     <disable_collisions link1="${link_prefix}base_link" link2="${link_prefix}link1" reason="Adjacent" />
-    <disable_collisions link1="${link_prefix}base_link" link2="${link_prefix}link2" reason="Never" />
-    <disable_collisions link1="${link_prefix}base_link" link2="${link_prefix}link3" reason="Never" />
     <disable_collisions link1="${link_prefix}link1" link2="${link_prefix}link2" reason="Adjacent" />
-    <disable_collisions link1="${link_prefix}link1" link2="${link_prefix}link3" reason="Never" />
     <disable_collisions link1="${link_prefix}link2" link2="${link_prefix}link3" reason="Adjacent" />
-    <disable_collisions link1="${link_prefix}link2" link2="${link_prefix}link4" reason="Never" />
     <disable_collisions link1="${link_prefix}link3" link2="${link_prefix}link4" reason="Adjacent" />
-    <disable_collisions link1="${link_prefix}link3" link2="${link_prefix}link5" reason="Never" />
-    <disable_collisions link1="${link_prefix}link3" link2="${link_prefix}link6" reason="Never" />
     <disable_collisions link1="${link_prefix}link4" link2="${link_prefix}link5" reason="Adjacent" />
-    <disable_collisions link1="${link_prefix}link4" link2="${link_prefix}link6" reason="Never" />
     <disable_collisions link1="${link_prefix}link5" link2="${link_prefix}link6" reason="Adjacent" />
-    <xacro:if value="$(eval arm_type == 'nero')">
-      <disable_collisions link1="${link_prefix}base_link" link2="${link_prefix}link4" reason="Never" />
-      <disable_collisions link1="${link_prefix}base_link" link2="${link_prefix}link5" reason="Never" />
-      <disable_collisions link1="${link_prefix}base_link" link2="${link_prefix}link6" reason="Never" />
-      <disable_collisions link1="${link_prefix}base_link" link2="${link_prefix}link7" reason="Never" />
-      <disable_collisions link1="${link_prefix}link1" link2="${link_prefix}link4" reason="Never" />
-      <disable_collisions link1="${link_prefix}link1" link2="${link_prefix}link5" reason="Never" />
-      <disable_collisions link1="${link_prefix}link1" link2="${link_prefix}link6" reason="Never" />
-      <disable_collisions link1="${link_prefix}link1" link2="${link_prefix}link7" reason="Never" />
-      <disable_collisions link1="${link_prefix}link2" link2="${link_prefix}link5" reason="Never" />
-      <disable_collisions link1="${link_prefix}link2" link2="${link_prefix}link6" reason="Never" />
-      <disable_collisions link1="${link_prefix}link2" link2="${link_prefix}link7" reason="Never" />
-      <disable_collisions link1="${link_prefix}link3" link2="${link_prefix}link7" reason="Never" />
-      <disable_collisions link1="${link_prefix}link4" link2="${link_prefix}link7" reason="Never" />
-      <disable_collisions link1="${link_prefix}link5" link2="${link_prefix}link7" reason="Never" />
-      <disable_collisions link1="${link_prefix}link6" link2="${link_prefix}link7" reason="Adjacent" />
+    <disable_collisions link1="${link_prefix}link6" link2="${link_prefix}link7" reason="Adjacent" />
+    <xacro:if value="${mount_body_link != ''}">
+      <disable_collisions link1="${mount_body_link}" link2="${link_prefix}base_link" reason="Adjacent" />
     </xacro:if>
   </xacro:macro>
@@ -98,5 +86,5 @@
       <joint name="${side}_pinky_pip_joint" />
     </group>
-    <end_effector name="${side}_omnihand_eef" parent_link="tcp_link" group="hand" parent_group="${planning_group_name}" />
+    <end_effector name="${side}_omnihand_eef" parent_link="${end_effector_parent_link}" group="hand" parent_group="${planning_group_name}" />
     <group_state name="hand_open" group="hand">
       <joint name="${side}_thumb_roll_joint" value="0.0" />
@@ -185,5 +173,5 @@
       <joint name="gripper_joint2" />
     </group>
-    <end_effector name="gripper_eef" parent_link="tcp_link" group="gripper" parent_group="${planning_group_name}" />
+    <end_effector name="gripper_eef" parent_link="${end_effector_parent_link}" group="gripper" parent_group="${planning_group_name}" />
     <group_state name="gripper_open" group="gripper">
       <joint name="gripper_joint1" value="0.05" />
@@ -236,5 +224,5 @@
       <link name="left_pinky_distal_link" />
     </group>
-    <end_effector name="left_hand_eef" parent_link="tcp_link" group="hand" parent_group="${planning_group_name}" />
+    <end_effector name="left_hand_eef" parent_link="${end_effector_parent_link}" group="hand" parent_group="${planning_group_name}" />
     <group_state name="hand_open" group="hand">
       <joint name="left_thumb_metacarpal_joint" value="0.0" />
@@ -381,5 +369,5 @@
       <link name="right_pinky_distal_link" />
     </group>
-    <end_effector name="right_hand_eef" parent_link="tcp_link" group="hand" parent_group="${planning_group_name}" />
+    <end_effector name="right_hand_eef" parent_link="${end_effector_parent_link}" group="hand" parent_group="${planning_group_name}" />
     <group_state name="hand_open" group="hand">
       <joint name="right_thumb_metacarpal_joint" value="0.0" />
@@ -537,9 +525,9 @@
   <!-- ======================== ARM DISABLE COLLISIONS ======================== -->
   <xacro:if value="$(arg include_dual_arm_groups)">
-    <xacro:nero_arm_disable_collisions link_prefix="${left_arm_link_prefix}" />
-    <xacro:nero_arm_disable_collisions link_prefix="${right_arm_link_prefix}" />
+    <xacro:nero_arm_disable_collisions link_prefix="${left_arm_link_prefix}" mount_body_link="${left_mount_body_link}" />
+    <xacro:nero_arm_disable_collisions link_prefix="${right_arm_link_prefix}" mount_body_link="${right_mount_body_link}" />
   </xacro:if>
   <xacro:unless value="$(arg include_dual_arm_groups)">
-    <xacro:nero_arm_disable_collisions link_prefix="${arm_link_prefix}" />
+    <xacro:nero_arm_disable_collisions link_prefix="${arm_link_prefix}" mount_body_link="${mount_body_link}" />
   </xacro:unless>
 </robot>

Commit message: fix(moveit): add setup assistant metadata and mounted-body collision disable
- Install .setup_assistant so moveit_configs_utils can infer SRDF/URDF paths
- Add collision disable for mounted arm link1 to prevent OMPL planning failures
- Fix xacro conditionals from $(eval ...) to ${ ... } syntax for proper evaluation
- Add xacro properties for effector_type, revo2_type, omnihand_type

File: src/agx_arm_moveit/config/agx_arm.srdf.xacro (robot description, xacro)
@@ -26,4 +26,8 @@
   <xacro:arg name="right_arm_link_prefix" default="right_arm_" />
   <xacro:property name="arm_type" value="$(arg arm_type)" />
+  <xacro:property name="effector_type" value="$(arg effector_type)" />
+  <xacro:property name="revo2_type" value="$(arg revo2_type)" />
+  <xacro:property name="omnihand_type" value="$(arg omnihand_type)" />
+  <xacro:property name="include_end_effector_groups" value="$(arg include_end_effector_groups)" />
   <xacro:property name="flange_link" value="${arm_link_prefix}link7" />
   <xacro:property name="planning_group_name" value="$(arg planning_group_name)" />
@@ -71,4 +75,5 @@
     <xacro:if value="${mount_body_link != ''}">
       <disable_collisions link1="${mount_body_link}" link2="${link_prefix}base_link" reason="Adjacent" />
+      <disable_collisions link1="${mount_body_link}" link2="${link_prefix}link1" reason="Adjacent" />
     </xacro:if>
   </xacro:macro>
@@ -165,5 +170,5 @@
   </xacro:unless>
   <!-- ======================== GRIPPER GROUP ======================== -->
-  <xacro:if value="$(eval include_end_effector_groups == 'true' and effector_type == 'agx_gripper')">
+  <xacro:if value="${str(include_end_effector_groups).lower() == 'true' and effector_type == 'agx_gripper'}">
     <group name="gripper">
       <link name="gripper_base" />
@@ -192,8 +197,8 @@
     <disable_collisions link1="gripper_link1" link2="${flange_link}" reason="Never" />
     <disable_collisions link1="gripper_link2" link2="${flange_link}" reason="Never" />
-    <xacro:unless value="$(eval arm_type == 'nero')">
+    <xacro:unless value="${arm_type == 'nero'}">
       <disable_collisions link1="gripper_base" link2="link5" reason="Never" />
     </xacro:unless>
-    <xacro:if value="$(eval arm_type == 'nero')">
+    <xacro:if value="${arm_type == 'nero'}">
       <disable_collisions link1="gripper_flange" link2="link7" reason="Adjacent" />
       <disable_collisions link1="gripper_flange" link2="gripper_base" reason="Adjacent" />
@@ -203,5 +208,5 @@
   </xacro:if>
   <!-- ======================== REVO2 LEFT HAND GROUP ======================== -->
-  <xacro:if value="$(eval include_end_effector_groups == 'true' and effector_type == 'revo2' and revo2_type == 'left')">
+  <xacro:if value="${str(include_end_effector_groups).lower() == 'true' and effector_type == 'revo2' and revo2_type == 'left'}">
     <group name="hand">
       <link name="left_base_link" />
@@ -348,5 +353,5 @@
   </xacro:if>
   <!-- ======================== REVO2 RIGHT HAND GROUP ======================== -->
-  <xacro:if value="$(eval include_end_effector_groups == 'true' and effector_type == 'revo2' and revo2_type == 'right')">
+  <xacro:if value="${str(include_end_effector_groups).lower() == 'true' and effector_type == 'revo2' and revo2_type == 'right'}">
     <group name="hand">
       <link name="right_base_link" />
@@ -493,8 +498,8 @@
   </xacro:if>
   <!-- ======================== OMNIHAND GROUP ======================== -->
-  <xacro:if value="$(eval include_end_effector_groups == 'true' and effector_type == 'omnihand' and omnihand_type == 'left')">
+  <xacro:if value="${str(include_end_effector_groups).lower() == 'true' and effector_type == 'omnihand' and omnihand_type == 'left'}">
     <xacro:omnihand_group side="left" />
   </xacro:if>
-  <xacro:if value="$(eval include_end_effector_groups == 'true' and effector_type == 'omnihand' and omnihand_type == 'right')">
+  <xacro:if value="${str(include_end_effector_groups).lower() == 'true' and effector_type == 'omnihand' and omnihand_type == 'right'}">
     <xacro:omnihand_group side="right" />
   </xacro:if>
