Commit message: feat(bringup): Add duo_hand bringup and execution profile.
- Wire downstream launches and arguments.
- Add srdf xacro and tests.

fix(bringup): Resolve wrong/quite fallback of a missing left arm to standard can (right arm) in duo_arm and left_hand settings. This caused the left arm use the right arm's feedback if no port detail is given.

File: src/agx_arm_moveit/config/agx_arm.srdf.xacro (robot description, xacro)
@@ -15,4 +15,8 @@
   <xacro:arg name="include_end_effector_groups" default="true" />
   <xacro:arg name="include_dual_arm_groups" default="false" />
+  <!-- Per-side OmniHand instantiation for the dual-arm slice (duo_hand profile);
+       ignored unless include_dual_arm_groups is true. -->
+  <xacro:arg name="include_left_omnihand" default="false" />
+  <xacro:arg name="include_right_omnihand" default="false" />
   <xacro:arg name="left_arm_base_frame" default="left_arm_base_link" />
   <xacro:arg name="left_arm_tip_frame" default="left_arm_nero_tool0" />
@@ -39,4 +43,6 @@
   <xacro:property name="arm_link_prefix" value="$(arg arm_link_prefix)" />
   <xacro:property name="include_dual_arm_groups" value="$(arg include_dual_arm_groups)" />
+  <xacro:property name="include_left_omnihand" value="$(arg include_left_omnihand)" />
+  <xacro:property name="include_right_omnihand" value="$(arg include_right_omnihand)" />
   <xacro:property name="left_arm_base_frame" value="$(arg left_arm_base_frame)" />
   <xacro:property name="left_arm_tip_frame" value="$(arg left_arm_tip_frame)" />
@@ -78,6 +84,14 @@
     </xacro:if>
   </xacro:macro>
-  <xacro:macro name="omnihand_group" params="side">
-    <group name="hand">
+  <!-- Per-side instantiable: the single-side profiles keep the legacy defaults
+       (group "hand", the file-level planning group / parent link / link prefix),
+       while the dual-arm slice instantiates it once per side with explicit
+       group_name/parent_group/parent_link/link_prefix so the two hands do not
+       collide on the MoveIt group name. -->
+  <xacro:macro name="omnihand_group" params="side group_name:='hand' parent_group:='' parent_link:='' link_prefix:=''">
+    <xacro:property name="resolved_parent_group" value="${parent_group if parent_group != '' else planning_group_name}" />
+    <xacro:property name="resolved_parent_link" value="${parent_link if parent_link != '' else end_effector_parent_link}" />
+    <xacro:property name="resolved_link_prefix" value="${link_prefix if link_prefix != '' else arm_link_prefix}" />
+    <group name="${group_name}">
       <joint name="${side}_thumb_roll_joint" />
       <joint name="${side}_thumb_abad_joint" />
@@ -93,6 +107,6 @@
       <joint name="${side}_pinky_mcp_joint" />
     </group>
-    <end_effector name="${side}_omnihand_eef" parent_link="${end_effector_parent_link}" group="hand" parent_group="${planning_group_name}" />
-    <group_state name="hand_open" group="hand">
+    <end_effector name="${side}_omnihand_eef" parent_link="${resolved_parent_link}" group="${group_name}" parent_group="${resolved_parent_group}" />
+    <group_state name="hand_open" group="${group_name}">
       <joint name="${side}_thumb_roll_joint" value="0.0" />
       <joint name="${side}_thumb_abad_joint" value="0.0" />
@@ -108,5 +122,5 @@
       <joint name="${side}_pinky_mcp_joint" value="0.0" />
     </group_state>
-    <group_state name="hand_half_close" group="hand">
+    <group_state name="hand_half_close" group="${group_name}">
       <joint name="${side}_thumb_roll_joint" value="${-0.2 if side == 'left' else 0.2}" />
       <joint name="${side}_thumb_abad_joint" value="${0.3 if side == 'left' else -0.3}" />
@@ -122,5 +136,5 @@
       <joint name="${side}_pinky_mcp_joint" value="0.6" />
     </group_state>
-    <group_state name="hand_close" group="hand">
+    <group_state name="hand_close" group="${group_name}">
       <joint name="${side}_thumb_roll_joint" value="${-0.4 if side == 'left' else 0.4}" />
       <joint name="${side}_thumb_abad_joint" value="${0.5 if side == 'left' else -0.5}" />
@@ -143,8 +157,8 @@
     <passive_joint name="${side}_pinky_pip_joint" />
     <passive_joint name="${side}_pinky_dip_joint" />
-    <disable_collisions link1="${arm_link_prefix}link7" link2="${arm_link_prefix}omnihand_flange" reason="Adjacent" />
-    <disable_collisions link1="${arm_link_prefix}link6" link2="${arm_link_prefix}omnihand_flange" reason="Never" />
-    <disable_collisions link1="${arm_link_prefix}omnihand_flange" link2="${side}_base_link" reason="Adjacent" />
-    <disable_collisions link1="${arm_link_prefix}omnihand_flange" link2="${side}_palm" reason="Adjacent" />
+    <disable_collisions link1="${resolved_link_prefix}link7" link2="${resolved_link_prefix}omnihand_flange" reason="Adjacent" />
+    <disable_collisions link1="${resolved_link_prefix}link6" link2="${resolved_link_prefix}omnihand_flange" reason="Never" />
+    <disable_collisions link1="${resolved_link_prefix}omnihand_flange" link2="${side}_base_link" reason="Adjacent" />
+    <disable_collisions link1="${resolved_link_prefix}omnihand_flange" link2="${side}_palm" reason="Adjacent" />
     <!-- Disable ALL intra-hand collision pairs. The hand joints are never planned
          by the arm groups (their values come from hardware readback), self-contact
@@ -490,4 +504,15 @@
       <group name="right_arm" />
     </group>
+    <!-- Per-side OmniHand groups for the dual-arm slice (duo_hand profile):
+         distinct group names + per-side parent group/link/prefix so the two
+         hands coexist, including each side's intra-hand collision ACM. -->
+    <xacro:if value="${str(include_left_omnihand).lower() == 'true'}">
+      <xacro:omnihand_group side="left" group_name="left_hand" parent_group="left_arm"
+                            parent_link="${left_arm_tip_frame}" link_prefix="${left_arm_link_prefix}" />
+    </xacro:if>
+    <xacro:if value="${str(include_right_omnihand).lower() == 'true'}">
+      <xacro:omnihand_group side="right" group_name="right_hand" parent_group="right_arm"
+                            parent_link="${right_arm_tip_frame}" link_prefix="${right_arm_link_prefix}" />
+    </xacro:if>
   </xacro:if>
   <xacro:unless value="$(arg include_dual_arm_groups)">

Commit message: feat(coordination): make tea_pour_duo_v2 a duo activity with taught-density replay
v1 drove the left side alone with the right merely live. v2 stages the right arm
into a support pose first, replays the two longest motions as both_arms takes
that were taught on both arms at once, and overlaps three arm moves with a hand
shape.

- Recorded actions reference lean sidecars under config/recordings/ instead of
  inlining waypoints, so the taught density the retiming needs survives and the
  side-prefixed joint names are checked against the planning group.
- Every arm action in a graph is now planned before the first one moves, anchor
  moves included: an anchor naming a pose that no longer exists used to fail at
  dispatch, with the arm mid-sequence and possibly holding the payload.
- A retryable MoveIt planning failure gets a fresh goal rather than another
  attempt inside the same one, which shares a goal sampler that has already
  failed.
- The right hand is out of service, so the activity commands it nowhere; its
  three actions stay defined so restoring them is an edge change.

Validation: package tests. The activity itself is unexercised end to end since
the right hand was withdrawn — the right arm's takes were taught with a shaped
hand and now replay with a flat one.

File: src/agx_arm_moveit/config/agx_arm.srdf.xacro (robot description, xacro)
@@ -82,4 +82,11 @@
       <disable_collisions link1="${mount_body_link}" link2="${link_prefix}base_link" reason="Adjacent" />
       <disable_collisions link1="${mount_body_link}" link2="${link_prefix}link1" reason="Adjacent" />
+      <!-- link2 rotates about the mount, so it sweeps along the torso hull by
+           construction: over the whole j1 x j2 range it never gets further than
+           12.9 mm (left) / 13.3 mm (right) from the body, median 7.2 / 8.0 mm.
+           A check on a pair that is always within 13 mm and touches at 0.01 mm
+           on a pose an operator back-drove the arm into by hand yields refusals,
+           not safety. Measured 2026-08-27, docs/control/bringups/tea_demo.md. -->
+      <disable_collisions link1="${mount_body_link}" link2="${link_prefix}link2" reason="Never" />
     </xacro:if>
   </xacro:macro>

File: src/agx_arm_sim/agx_arm_description/agx_arm_urdf/nero/urdf/nero_with_left_omnihand_description.xacro (robot description, xacro)
@@ -4,5 +4,5 @@
   <xacro:include filename="$(find agx_arm_description)/agx_arm_urdf/nero/urdf/nero_with_omnihand_flange_description.xacro"/>
   <joint name="hand_base_joint" type="fixed">
-    <origin xyz="0.0 0.0 0.012" rpy="0 0 3.1415926"/>
+    <origin xyz="0.0 0.0 0.005" rpy="0 0 3.1415926"/>
     <parent link="omnihand_flange"/>
     <child link="left_base_link"/>

File: src/agx_arm_sim/agx_arm_description/agx_arm_urdf/nero/urdf/nero_with_right_omnihand_description.xacro (robot description, xacro)
@@ -4,5 +4,5 @@
   <xacro:include filename="$(find agx_arm_description)/agx_arm_urdf/nero/urdf/nero_with_omnihand_flange_description.xacro"/>
   <joint name="hand_base_joint" type="fixed">
-    <origin xyz="0.0 0.0 0.012" rpy="0 0 3.1415926"/>
+    <origin xyz="0.0 0.0 0.005" rpy="0 0 3.1415926"/>
     <parent link="omnihand_flange"/>
     <child link="right_base_link"/>

File: src/duo_body_description/urdf/duo_body.xacro (robot description, xacro)
@@ -22,5 +22,6 @@
       <child link="left_arm_mount_link"/>
       <!--<origin xyz="-0.137511 0.104055 0.070000" rpy="0 1.570796 -0.837758"/>-->
-      <origin xyz="-0.154602 0.110059 0.078262" rpy="0 -1.570796 -0.837758"/>
+      <!--origin xyz="-0.154602 0.110059 0.078262" rpy="0 -1.570796 -0.837758"/-->
+      <origin xyz="-0.1370 0.10059 0.071262" rpy="0 -1.570796 -0.737758"/>
     </joint>
     <link name="right_arm_mount_link"/>
@@ -29,5 +30,5 @@
       <child link="right_arm_mount_link"/>
       <!--<origin xyz="0.137511 0.104055 0.070000" rpy="0 1.570796 0.837758"/>-->
-      <origin xyz="0.154602 0.110059 0.071262" rpy="0 1.570796 0.837758"/>
+      <origin xyz="0.1370 0.10059 0.071262" rpy="0 1.570796 0.737758"/>
     </joint>
   </xacro:macro>

File: src/duo_body_description/urdf/nero_arm_macro.xacro (robot description, xacro)
@@ -257,5 +257,5 @@
       </link>
       <joint name="${arm_prefix}left_hand_base_joint" type="fixed">
-        <origin xyz="0.0 0.0 0.012" rpy="0 0 3.1415926"/>
+        <origin xyz="0.0 0.0 0.005" rpy="0 0 3.1415926"/>
         <parent link="${arm_prefix}omnihand_flange"/>
         <child link="left_base_link"/>
@@ -281,5 +281,5 @@
       </link>
       <joint name="${arm_prefix}right_hand_base_joint" type="fixed">
-        <origin xyz="0.0 0.0 0.012" rpy="0 0 3.1415926"/>
+        <origin xyz="0.0 0.0 0.005" rpy="0 0 3.1415926"/>
         <parent link="${arm_prefix}omnihand_flange"/>
         <child link="right_base_link"/>

Commit message: feat(moveit): make the gripper a per-side end effector, both arms
The gripper's SRDF group named its links and joints without a prefix, so a
prefixed model got a group pointing at links that do not exist, and only one arm
could ever carry one.

- The group is now instantiable per side, like the OmniHand's, with its own
  group name, parent group, parent link and prefixes. Both arms can carry a
  gripper; the single-arm case is the macro's default and is unchanged.
- A gripper has no side of its own, so the side comes from the joint prefix of
  the arm instance it is mounted on rather than from a type field.
- both_arms accepts agx_gripper as a result; the runtime contract test now
  guards revo2 as the rejected case and the gripper as an accepted one.
- Gripper fingers get prismatic planning limits in metres: 3.0 m/s from the
  URDF, with 2.5 * v_max as the acceleration stand-in, marked as such. MoveIt
  was falling back to 1 rad/s^2 for them.
- New presets left_gripper, right_gripper and duo_gripper.

Only the right arm carries a gripper today; the left and duo presets are
structurally complete and unvalidated on hardware.

Validation: package tests, plus cross-checking every SRDF link and joint
reference against the generated URDF for the prefixed, unprefixed and dual
cases. MoveIt plans the gripper group but cannot execute it — no controller
actuates those joints yet.

File: src/agx_arm_moveit/config/agx_arm.srdf.xacro (robot description, xacro)
@@ -19,4 +19,6 @@
   <xacro:arg name="include_left_omnihand" default="false" />
   <xacro:arg name="include_right_omnihand" default="false" />
+  <xacro:arg name="include_left_gripper" default="false" />
+  <xacro:arg name="include_right_gripper" default="false" />
   <xacro:arg name="left_arm_base_frame" default="left_arm_base_link" />
   <xacro:arg name="left_arm_tip_frame" default="left_arm_nero_tool0" />
@@ -45,4 +47,6 @@
   <xacro:property name="include_left_omnihand" value="$(arg include_left_omnihand)" />
   <xacro:property name="include_right_omnihand" value="$(arg include_right_omnihand)" />
+  <xacro:property name="include_left_gripper" value="$(arg include_left_gripper)" />
+  <xacro:property name="include_right_gripper" value="$(arg include_right_gripper)" />
   <xacro:property name="left_arm_base_frame" value="$(arg left_arm_base_frame)" />
   <xacro:property name="left_arm_tip_frame" value="$(arg left_arm_tip_frame)" />
@@ -541,40 +545,57 @@
   </xacro:unless>
   <!-- ======================== GRIPPER GROUP ======================== -->
+  <!-- Per-side instantiable, like omnihand_group: distinct group name plus its
+       own parent group/link and link/joint prefixes, so both arms can carry a
+       gripper in the dual-arm slice. Defaults reproduce the single-arm case. -->
+  <xacro:macro name="agx_gripper_group"
+               params="group_name:='gripper' eef_name:='gripper_eef' parent_group:='' parent_link:='' link_prefix:='' joint_prefix:=''">
+    <xacro:property name="g_parent_group" value="${parent_group if parent_group != '' else planning_group_name}" />
+    <xacro:property name="g_parent_link" value="${parent_link if parent_link != '' else end_effector_parent_link}" />
+    <xacro:property name="g_link_prefix" value="${link_prefix if link_prefix != '' else arm_link_prefix}" />
+    <xacro:property name="g_joint_prefix" value="${joint_prefix if joint_prefix != '' else arm_joint_prefix}" />
+    <group name="${group_name}">
+      <link name="${g_link_prefix}gripper_base" />
+      <link name="${g_link_prefix}gripper_link1" />
+      <link name="${g_link_prefix}gripper_link2" />
+      <joint name="${g_joint_prefix}gripper_joint1" />
+      <joint name="${g_joint_prefix}gripper_joint2" />
+    </group>
+    <end_effector name="${eef_name}" parent_link="${g_parent_link}" group="${group_name}" parent_group="${g_parent_group}" />
+    <group_state name="${group_name}_open" group="${group_name}">
+      <joint name="${g_joint_prefix}gripper_joint1" value="0.05" />
+      <joint name="${g_joint_prefix}gripper_joint2" value="-0.05" />
+    </group_state>
+    <group_state name="${group_name}_half" group="${group_name}">
+      <joint name="${g_joint_prefix}gripper_joint1" value="0.025" />
+      <joint name="${g_joint_prefix}gripper_joint2" value="-0.025" />
+    </group_state>
+    <group_state name="${group_name}_close" group="${group_name}">
+      <joint name="${g_joint_prefix}gripper_joint1" value="0.0" />
+      <joint name="${g_joint_prefix}gripper_joint2" value="0.0" />
+    </group_state>
+    <disable_collisions link1="${g_link_prefix}gripper_base" link2="${g_link_prefix}link7" reason="Adjacent" />
+    <disable_collisions link1="${g_link_prefix}gripper_base" link2="${g_link_prefix}gripper_link1" reason="Adjacent" />
+    <disable_collisions link1="${g_link_prefix}gripper_base" link2="${g_link_prefix}gripper_link2" reason="Adjacent" />
+    <disable_collisions link1="${g_link_prefix}gripper_link1" link2="${g_link_prefix}gripper_link2" reason="Adjacent" />
+    <disable_collisions link1="${g_link_prefix}gripper_link1" link2="${g_link_prefix}link7" reason="Never" />
+    <disable_collisions link1="${g_link_prefix}gripper_link2" link2="${g_link_prefix}link7" reason="Never" />
+    <disable_collisions link1="${g_link_prefix}gripper_flange" link2="${g_link_prefix}link7" reason="Adjacent" />
+    <disable_collisions link1="${g_link_prefix}gripper_flange" link2="${g_link_prefix}gripper_base" reason="Adjacent" />
+    <disable_collisions link1="${g_link_prefix}gripper_flange" link2="${g_link_prefix}link6" reason="Never" />
+    <disable_collisions link1="${g_link_prefix}gripper_base" link2="${g_link_prefix}link6" reason="Never" />
+  </xacro:macro>
+  <!-- Per-side gripper groups for the dual-arm slice (duo_gripper profile). -->
+  <xacro:if value="${str(include_left_gripper).lower() == 'true'}">
+    <xacro:agx_gripper_group group_name="left_gripper" eef_name="left_gripper_eef" parent_group="left_arm"
+                             parent_link="${left_arm_tip_frame}"
+                             link_prefix="${left_arm_link_prefix}" joint_prefix="${left_arm_joint_prefix}" />
+  </xacro:if>
+  <xacro:if value="${str(include_right_gripper).lower() == 'true'}">
+    <xacro:agx_gripper_group group_name="right_gripper" eef_name="right_gripper_eef" parent_group="right_arm"
+                             parent_link="${right_arm_tip_frame}"
+                             link_prefix="${right_arm_link_prefix}" joint_prefix="${right_arm_joint_prefix}" />
+  </xacro:if>
   <xacro:if value="${str(include_end_effector_groups).lower() == 'true' and effector_type == 'agx_gripper'}">
-    <group name="gripper">
-      <link name="gripper_base" />
-      <link name="gripper_link1" />
-      <link name="gripper_link2" />
-      <joint name="gripper_joint1" />
-      <joint name="gripper_joint2" />
-    </group>
-    <end_effector name="gripper_eef" parent_link="${end_effector_parent_link}" group="gripper" parent_group="${planning_group_name}" />
-    <group_state name="gripper_open" group="gripper">
-      <joint name="gripper_joint1" value="0.05" />
-      <joint name="gripper_joint2" value="-0.05" />
-    </group_state>
-    <group_state name="gripper_half" group="gripper">
-      <joint name="gripper_joint1" value="0.025" />
-      <joint name="gripper_joint2" value="-0.025" />
-    </group_state>
-    <group_state name="gripper_close" group="gripper">
-      <joint name="gripper_joint1" value="0.0" />
-      <joint name="gripper_joint2" value="0.0" />
-    </group_state>
-    <disable_collisions link1="gripper_base" link2="${flange_link}" reason="Adjacent" />
-    <disable_collisions link1="gripper_base" link2="gripper_link1" reason="Adjacent" />
-    <disable_collisions link1="gripper_base" link2="gripper_link2" reason="Adjacent" />
-    <disable_collisions link1="gripper_link1" link2="gripper_link2" reason="Adjacent" />
-    <disable_collisions link1="gripper_link1" link2="${flange_link}" reason="Never" />
-    <disable_collisions link1="gripper_link2" link2="${flange_link}" reason="Never" />
-    <xacro:unless value="${arm_type == 'nero'}">
-      <disable_collisions link1="gripper_base" link2="link5" reason="Never" />
-    </xacro:unless>
-    <xacro:if value="${arm_type == 'nero'}">
-      <disable_collisions link1="gripper_flange" link2="link7" reason="Adjacent" />
-      <disable_collisions link1="gripper_flange" link2="gripper_base" reason="Adjacent" />
-      <disable_collisions link1="gripper_flange" link2="link6" reason="Never" />
-      <disable_collisions link1="gripper_base" link2="link6" reason="Never" />
-    </xacro:if>
+    <xacro:agx_gripper_group />
   </xacro:if>
   <!-- ======================== REVO2 LEFT HAND GROUP ======================== -->
