Commit message: feat(omnihand): add simulation-first moveit integration
Add the first repo-owned OmniHand simulation path across agx_arm_description and agx_arm_moveit while keeping hardware transport and runtime bring-up explicitly out of scope.

- normalize left/right OmniHand description assets into the canonical agx_arm_description package

- expose OmniHand through display.launch.py, display_control.launch.py, and MoveIt effector_type:=omnihand

- add mock ros2_control joints, MoveIt controller profiles, and SRDF hand groups for left/right simulation

File: src/agx_arm_moveit/config/agx_arm.ros2_control.xacro (robot description, xacro)
@@ -1,5 +1,5 @@
 <?xml version="1.0"?>
 <robot xmlns:xacro="http://www.ros.org/wiki/xacro">
-  <xacro:macro name="agx_arm_ros2_control" params="name initial_positions_file arm_type effector_type revo2_type">
+  <xacro:macro name="agx_arm_ros2_control" params="name initial_positions_file arm_type effector_type revo2_type omnihand_type">
     <xacro:property name="initial_positions" value="${xacro.load_yaml(initial_positions_file)['initial_positions']}" />
     <ros2_control name="${name}" type="system">
@@ -90,4 +90,28 @@
         <joint name="right_pinky_proximal_joint"><command_interface name="position" /><state_interface name="position"><param name="initial_value">${initial_positions['right_pinky_proximal_joint']}</param></state_interface><state_interface name="velocity" /></joint>
       </xacro:if>
+      <xacro:if value="${effector_type == 'omnihand' and omnihand_type == 'left'}">
+        <joint name="left_thumb_roll_joint"><command_interface name="position" /><state_interface name="position"><param name="initial_value">${initial_positions['left_thumb_roll_joint']}</param></state_interface><state_interface name="velocity" /></joint>
+        <joint name="left_thumb_abad_joint"><command_interface name="position" /><state_interface name="position"><param name="initial_value">${initial_positions['left_thumb_abad_joint']}</param></state_interface><state_interface name="velocity" /></joint>
+        <joint name="left_thumb_mcp_joint"><command_interface name="position" /><state_interface name="position"><param name="initial_value">${initial_positions['left_thumb_mcp_joint']}</param></state_interface><state_interface name="velocity" /></joint>
+        <joint name="left_index_abad_joint"><command_interface name="position" /><state_interface name="position"><param name="initial_value">${initial_positions['left_index_abad_joint']}</param></state_interface><state_interface name="velocity" /></joint>
+        <joint name="left_index_pip_joint"><command_interface name="position" /><state_interface name="position"><param name="initial_value">${initial_positions['left_index_pip_joint']}</param></state_interface><state_interface name="velocity" /></joint>
+        <joint name="left_middle_pip_joint"><command_interface name="position" /><state_interface name="position"><param name="initial_value">${initial_positions['left_middle_pip_joint']}</param></state_interface><state_interface name="velocity" /></joint>
+        <joint name="left_ring_abad_joint"><command_interface name="position" /><state_interface name="position"><param name="initial_value">${initial_positions['left_ring_abad_joint']}</param></state_interface><state_interface name="velocity" /></joint>
+        <joint name="left_ring_pip_joint"><command_interface name="position" /><state_interface name="position"><param name="initial_value">${initial_positions['left_ring_pip_joint']}</param></state_interface><state_interface name="velocity" /></joint>
+        <joint name="left_pinky_abad_joint"><command_interface name="position" /><state_interface name="position"><param name="initial_value">${initial_positions['left_pinky_abad_joint']}</param></state_interface><state_interface name="velocity" /></joint>
+        <joint name="left_pinky_pip_joint"><command_interface name="position" /><state_interface name="position"><param name="initial_value">${initial_positions['left_pinky_pip_joint']}</param></state_interface><state_interface name="velocity" /></joint>
+      </xacro:if>
+      <xacro:if value="${effector_type == 'omnihand' and omnihand_type == 'right'}">
+        <joint name="right_thumb_roll_joint"><command_interface name="position" /><state_interface name="position"><param name="initial_value">${initial_positions['right_thumb_roll_joint']}</param></state_interface><state_interface name="velocity" /></joint>
+        <joint name="right_thumb_abad_joint"><command_interface name="position" /><state_interface name="position"><param name="initial_value">${initial_positions['right_thumb_abad_joint']}</param></state_interface><state_interface name="velocity" /></joint>
+        <joint name="right_thumb_mcp_joint"><command_interface name="position" /><state_interface name="position"><param name="initial_value">${initial_positions['right_thumb_mcp_joint']}</param></state_interface><state_interface name="velocity" /></joint>
+        <joint name="right_index_abad_joint"><command_interface name="position" /><state_interface name="position"><param name="initial_value">${initial_positions['right_index_abad_joint']}</param></state_interface><state_interface name="velocity" /></joint>
+        <joint name="right_index_pip_joint"><command_interface name="position" /><state_interface name="position"><param name="initial_value">${initial_positions['right_index_pip_joint']}</param></state_interface><state_interface name="velocity" /></joint>
+        <joint name="right_middle_pip_joint"><command_interface name="position" /><state_interface name="position"><param name="initial_value">${initial_positions['right_middle_pip_joint']}</param></state_interface><state_interface name="velocity" /></joint>
+        <joint name="right_ring_abad_joint"><command_interface name="position" /><state_interface name="position"><param name="initial_value">${initial_positions['right_ring_abad_joint']}</param></state_interface><state_interface name="velocity" /></joint>
+        <joint name="right_ring_pip_joint"><command_interface name="position" /><state_interface name="position"><param name="initial_value">${initial_positions['right_ring_pip_joint']}</param></state_interface><state_interface name="velocity" /></joint>
+        <joint name="right_pinky_abad_joint"><command_interface name="position" /><state_interface name="position"><param name="initial_value">${initial_positions['right_pinky_abad_joint']}</param></state_interface><state_interface name="velocity" /></joint>
+        <joint name="right_pinky_pip_joint"><command_interface name="position" /><state_interface name="position"><param name="initial_value">${initial_positions['right_pinky_pip_joint']}</param></state_interface><state_interface name="velocity" /></joint>
+      </xacro:if>
     </ros2_control>
   </xacro:macro>

File: src/agx_arm_moveit/config/agx_arm.srdf.xacro (robot description, xacro)
@@ -4,6 +4,86 @@
   <xacro:arg name="effector_type" default="none" />
   <xacro:arg name="revo2_type" default="left" />
+  <xacro:arg name="omnihand_type" default="left" />
   <xacro:property name="arm_type" value="$(arg arm_type)" />
   <xacro:property name="flange_link" value="link7" />
+  <xacro:macro name="omnihand_group" params="side">
+    <group name="hand">
+      <joint name="${side}_thumb_roll_joint" />
+      <joint name="${side}_thumb_abad_joint" />
+      <joint name="${side}_thumb_mcp_joint" />
+      <joint name="${side}_index_abad_joint" />
+      <joint name="${side}_index_pip_joint" />
+      <joint name="${side}_middle_pip_joint" />
+      <joint name="${side}_ring_abad_joint" />
+      <joint name="${side}_ring_pip_joint" />
+      <joint name="${side}_pinky_abad_joint" />
+      <joint name="${side}_pinky_pip_joint" />
+    </group>
+    <end_effector name="${side}_omnihand_eef" parent_link="tcp_link" group="hand" parent_group="arm" />
+    <group_state name="hand_open" group="hand">
+      <joint name="${side}_thumb_roll_joint" value="0.0" />
+      <joint name="${side}_thumb_abad_joint" value="0.0" />
+      <joint name="${side}_thumb_mcp_joint" value="0.0" />
+      <joint name="${side}_index_abad_joint" value="0.0" />
+      <joint name="${side}_index_pip_joint" value="0.0" />
+      <joint name="${side}_middle_pip_joint" value="0.0" />
+      <joint name="${side}_ring_abad_joint" value="0.0" />
+      <joint name="${side}_ring_pip_joint" value="0.0" />
+      <joint name="${side}_pinky_abad_joint" value="0.0" />
+      <joint name="${side}_pinky_pip_joint" value="0.0" />
+    </group_state>
+    <group_state name="hand_half_close" group="hand">
+      <joint name="${side}_thumb_roll_joint" value="${-0.25 if side == 'left' else 0.25}" />
+      <joint name="${side}_thumb_abad_joint" value="${0.6 if side == 'left' else -0.6}" />
+      <joint name="${side}_thumb_mcp_joint" value="${-0.35 if side == 'left' else 0.35}" />
+      <joint name="${side}_index_abad_joint" value="${0.05 if side == 'left' else -0.05}" />
+      <joint name="${side}_index_pip_joint" value="0.7" />
+      <joint name="${side}_middle_pip_joint" value="0.7" />
+      <joint name="${side}_ring_abad_joint" value="${-0.05 if side == 'left' else 0.05}" />
+      <joint name="${side}_ring_pip_joint" value="0.7" />
+      <joint name="${side}_pinky_abad_joint" value="${-0.05 if side == 'left' else 0.05}" />
+      <joint name="${side}_pinky_pip_joint" value="0.7" />
+    </group_state>
+    <group_state name="hand_close" group="hand">
+      <joint name="${side}_thumb_roll_joint" value="${-0.45 if side == 'left' else 0.45}" />
+      <joint name="${side}_thumb_abad_joint" value="${1.0 if side == 'left' else -1.0}" />
+      <joint name="${side}_thumb_mcp_joint" value="${-0.6 if side == 'left' else 0.6}" />
+      <joint name="${side}_index_abad_joint" value="${0.1 if side == 'left' else -0.1}" />
+      <joint name="${side}_index_pip_joint" value="1.2" />
+      <joint name="${side}_middle_pip_joint" value="1.2" />
+      <joint name="${side}_ring_abad_joint" value="${-0.1 if side == 'left' else 0.1}" />
+      <joint name="${side}_ring_pip_joint" value="1.2" />
+      <joint name="${side}_pinky_abad_joint" value="${-0.1 if side == 'left' else 0.1}" />
+      <joint name="${side}_pinky_pip_joint" value="1.2" />
+    </group_state>
+    <passive_joint name="${side}_thumb_pip_joint" />
+    <passive_joint name="${side}_thumb_dip_joint" />
+    <passive_joint name="${side}_index_dip_joint" />
+    <passive_joint name="${side}_middle_dip_joint" />
+    <passive_joint name="${side}_ring_dip_joint" />
+    <passive_joint name="${side}_pinky_dip_joint" />
+    <disable_collisions link1="link7" link2="omnihand_flange" reason="Adjacent" />
+    <disable_collisions link1="link6" link2="omnihand_flange" reason="Never" />
+    <disable_collisions link1="omnihand_flange" link2="${side}_base_link" reason="Adjacent" />
+    <disable_collisions link1="omnihand_flange" link2="${side}_palm" reason="Adjacent" />
+    <disable_collisions link1="${side}_base_link" link2="${side}_palm" reason="Adjacent" />
+    <disable_collisions link1="${side}_palm" link2="${side}_thumb_roll" reason="Adjacent" />
+    <disable_collisions link1="${side}_palm" link2="${side}_index_abad" reason="Adjacent" />
+    <disable_collisions link1="${side}_palm" link2="${side}_middle_abad" reason="Adjacent" />
+    <disable_collisions link1="${side}_palm" link2="${side}_ring_abad" reason="Adjacent" />
+    <disable_collisions link1="${side}_palm" link2="${side}_pinky_abad" reason="Adjacent" />
+    <disable_collisions link1="${side}_thumb_roll" link2="${side}_thumb_abad" reason="Adjacent" />
+    <disable_collisions link1="${side}_thumb_abad" link2="${side}_thumb_mcp" reason="Adjacent" />
+    <disable_collisions link1="${side}_thumb_mcp" link2="${side}_thumb_pip" reason="Adjacent" />
+    <disable_collisions link1="${side}_thumb_pip" link2="${side}_thumb_dip" reason="Adjacent" />
+    <disable_collisions link1="${side}_index_abad" link2="${side}_index_pip" reason="Adjacent" />
+    <disable_collisions link1="${side}_index_pip" link2="${side}_index_dip" reason="Adjacent" />
+    <disable_collisions link1="${side}_middle_abad" link2="${side}_middle_pip" reason="Adjacent" />
+    <disable_collisions link1="${side}_middle_pip" link2="${side}_middle_dip" reason="Adjacent" />
+    <disable_collisions link1="${side}_ring_abad" link2="${side}_ring_pip" reason="Adjacent" />
+    <disable_collisions link1="${side}_ring_pip" link2="${side}_ring_dip" reason="Adjacent" />
+    <disable_collisions link1="${side}_pinky_abad" link2="${side}_pinky_pip" reason="Adjacent" />
+    <disable_collisions link1="${side}_pinky_pip" link2="${side}_pinky_dip" reason="Adjacent" />
+  </xacro:macro>
   <!-- ======================== ARM GROUP ======================== -->
   <group name="arm">
@@ -338,4 +418,11 @@
     </xacro:unless>
   </xacro:if>
+  <!-- ======================== OMNIHAND GROUP ======================== -->
+  <xacro:if value="$(eval effector_type == 'omnihand' and omnihand_type == 'left')">
+    <xacro:omnihand_group side="left" />
+  </xacro:if>
+  <xacro:if value="$(eval effector_type == 'omnihand' and omnihand_type == 'right')">
+    <xacro:omnihand_group side="right" />
+  </xacro:if>
   <!-- ======================== HOME STATE ======================== -->
   <xacro:unless value="$(eval arm_type == 'nero')">

File: src/agx_arm_moveit/config/agx_arm.urdf.xacro (robot description, xacro)
@@ -4,4 +4,5 @@
   <xacro:arg name="effector_type" default="none" />
   <xacro:arg name="revo2_type" default="left" />
+  <xacro:arg name="omnihand_type" default="left" />
   <xacro:arg name="initial_positions_file" default="initial_positions.yaml" />
   <xacro:arg name="tcp_offset_xyz" default="0 0 0" />
@@ -17,4 +18,10 @@
   <xacro:if value="$(eval effector_type == 'revo2' and revo2_type == 'right')">
     <xacro:include filename="$(find agx_arm_description)/agx_arm_urdf/$(arg arm_type)/urdf/$(arg arm_type)_with_right_revo2_description.xacro" />
+  </xacro:if>
+  <xacro:if value="$(eval effector_type == 'omnihand' and omnihand_type == 'left')">
+    <xacro:include filename="$(find agx_arm_description)/agx_arm_urdf/$(arg arm_type)/urdf/$(arg arm_type)_with_left_omnihand_description.xacro" />
+  </xacro:if>
+  <xacro:if value="$(eval effector_type == 'omnihand' and omnihand_type == 'right')">
+    <xacro:include filename="$(find agx_arm_description)/agx_arm_urdf/$(arg arm_type)/urdf/$(arg arm_type)_with_right_omnihand_description.xacro" />
   </xacro:if>
   <xacro:if value="$(eval effector_type == 'none')">
@@ -35,4 +42,5 @@
     effector_type="$(arg effector_type)"
     revo2_type="$(arg revo2_type)"
+    omnihand_type="$(arg omnihand_type)"
   />
 </robot>

File: src/agx_arm_sim/agx_arm_description/urdf/agx_arm_description.urdf.xacro (robot description, xacro)
@@ -8,5 +8,5 @@
     arm_type          : nero（当前工作区活动配置）
                         默认: nero
-    end_effector      : none | gripper | revo2_left | revo2_right
+    end_effector      : none | gripper | revo2_left | revo2_right | omnihand_left | omnihand_right
                         默认: none
     revo2_side        : left | right
@@ -22,4 +22,5 @@
     xacro agx_arm_description.urdf.xacro arm_type:=nero with_camera_stand:=true with_camera:=true
     xacro agx_arm_description.urdf.xacro arm_type:=nero end_effector:=revo2_right
+    xacro agx_arm_description.urdf.xacro arm_type:=nero end_effector:=omnihand_left
 -->
 <robot xmlns:xacro="http://www.ros.org/wiki/xacro" name="agx_arm">
@@ -197,4 +198,10 @@
     <xacro:if value="${ee == 'revo2_right'}">
       <xacro:include filename="${urdf_root}/nero/urdf/nero_with_right_revo2_description.xacro"/>
+    </xacro:if>
+    <xacro:if value="${ee == 'omnihand_left'}">
+      <xacro:include filename="${urdf_root}/nero/urdf/nero_with_left_omnihand_description.xacro"/>
+    </xacro:if>
+    <xacro:if value="${ee == 'omnihand_right'}">
+      <xacro:include filename="${urdf_root}/nero/urdf/nero_with_right_omnihand_description.xacro"/>
     </xacro:if>
     <xacro:if value="${ee == 'teach'}">
