Commit message: feat(omnihand,moveit): migrate hand description to OmniHand Pro O12 (12 active DoF)
Replace the legacy O10 OmniHand kinematic description with the official AgibotTech
OmniHand Pro O12 description (o12_hand_description-o12_t3, Mulan PSL v2), imported into
agx_arm_description as omnihand/urdf/xacro_pro + omnihand/meshes_pro. The vendor xacro
(const/material/thumb/index/middle/ring_pinky) is verbatim; hand.xacro is adapted to the
repo seam (macro `hand name mirror *origin`, palm parented to ${name}_base_link,
mirror_mesh derived from mirror, repo-local paths). The three includes that pulled the old
O10 hand.xacro now point at xacro_pro/hand.xacro.

Bring the MoveIt surfaces to the 12 active joints (thumb roll/abad/mcp/pip, index+middle
abad/mcp/pip, ring_mcp, pinky_mcp) so move_group models the real hand: SRDF omnihand_group
(joints, group_states, passive/mimic joints, O12 link collisions), the omnihand FJT
controller lists, initial_positions, and ros2_control. This fixes the components.launch
"Joint 'right_*_mcp_joint' not found in model 'duo_nero_system'" errors.

Validated on the arm64 host: agx_arm_description/agx_arm_moveit build clean; the standalone
and duo URDFs expand; and an offline cross-check of the expanded SRDF vs URDF reports every
SRDF joint/link resolving in the model (0 missing). Calibrated grasp/open presets and live
RViz/hardware confirmation remain follow-ups.

File: src/agx_arm_moveit/config/agx_arm.ros2_control.xacro (robot description, xacro)
@@ -94,11 +94,13 @@
         <joint name="left_thumb_abad_joint"><command_interface name="position" /><state_interface name="position"><param name="initial_value">${initial_positions['left_thumb_abad_joint']}</param></state_interface><state_interface name="velocity" /></joint>
         <joint name="left_thumb_mcp_joint"><command_interface name="position" /><state_interface name="position"><param name="initial_value">${initial_positions['left_thumb_mcp_joint']}</param></state_interface><state_interface name="velocity" /></joint>
+        <joint name="left_thumb_pip_joint"><command_interface name="position" /><state_interface name="position"><param name="initial_value">${initial_positions['left_thumb_pip_joint']}</param></state_interface><state_interface name="velocity" /></joint>
         <joint name="left_index_abad_joint"><command_interface name="position" /><state_interface name="position"><param name="initial_value">${initial_positions['left_index_abad_joint']}</param></state_interface><state_interface name="velocity" /></joint>
+        <joint name="left_index_mcp_joint"><command_interface name="position" /><state_interface name="position"><param name="initial_value">${initial_positions['left_index_mcp_joint']}</param></state_interface><state_interface name="velocity" /></joint>
         <joint name="left_index_pip_joint"><command_interface name="position" /><state_interface name="position"><param name="initial_value">${initial_positions['left_index_pip_joint']}</param></state_interface><state_interface name="velocity" /></joint>
+        <joint name="left_middle_abad_joint"><command_interface name="position" /><state_interface name="position"><param name="initial_value">${initial_positions['left_middle_abad_joint']}</param></state_interface><state_interface name="velocity" /></joint>
+        <joint name="left_middle_mcp_joint"><command_interface name="position" /><state_interface name="position"><param name="initial_value">${initial_positions['left_middle_mcp_joint']}</param></state_interface><state_interface name="velocity" /></joint>
         <joint name="left_middle_pip_joint"><command_interface name="position" /><state_interface name="position"><param name="initial_value">${initial_positions['left_middle_pip_joint']}</param></state_interface><state_interface name="velocity" /></joint>
-        <joint name="left_ring_abad_joint"><command_interface name="position" /><state_interface name="position"><param name="initial_value">${initial_positions['left_ring_abad_joint']}</param></state_interface><state_interface name="velocity" /></joint>
-        <joint name="left_ring_pip_joint"><command_interface name="position" /><state_interface name="position"><param name="initial_value">${initial_positions['left_ring_pip_joint']}</param></state_interface><state_interface name="velocity" /></joint>
-        <joint name="left_pinky_abad_joint"><command_interface name="position" /><state_interface name="position"><param name="initial_value">${initial_positions['left_pinky_abad_joint']}</param></state_interface><state_interface name="velocity" /></joint>
-        <joint name="left_pinky_pip_joint"><command_interface name="position" /><state_interface name="position"><param name="initial_value">${initial_positions['left_pinky_pip_joint']}</param></state_interface><state_interface name="velocity" /></joint>
+        <joint name="left_ring_mcp_joint"><command_interface name="position" /><state_interface name="position"><param name="initial_value">${initial_positions['left_ring_mcp_joint']}</param></state_interface><state_interface name="velocity" /></joint>
+        <joint name="left_pinky_mcp_joint"><command_interface name="position" /><state_interface name="position"><param name="initial_value">${initial_positions['left_pinky_mcp_joint']}</param></state_interface><state_interface name="velocity" /></joint>
       </xacro:if>
       <xacro:if value="${effector_type == 'omnihand' and omnihand_type == 'right'}">
@@ -106,11 +108,13 @@
         <joint name="right_thumb_abad_joint"><command_interface name="position" /><state_interface name="position"><param name="initial_value">${initial_positions['right_thumb_abad_joint']}</param></state_interface><state_interface name="velocity" /></joint>
         <joint name="right_thumb_mcp_joint"><command_interface name="position" /><state_interface name="position"><param name="initial_value">${initial_positions['right_thumb_mcp_joint']}</param></state_interface><state_interface name="velocity" /></joint>
+        <joint name="right_thumb_pip_joint"><command_interface name="position" /><state_interface name="position"><param name="initial_value">${initial_positions['right_thumb_pip_joint']}</param></state_interface><state_interface name="velocity" /></joint>
         <joint name="right_index_abad_joint"><command_interface name="position" /><state_interface name="position"><param name="initial_value">${initial_positions['right_index_abad_joint']}</param></state_interface><state_interface name="velocity" /></joint>
+        <joint name="right_index_mcp_joint"><command_interface name="position" /><state_interface name="position"><param name="initial_value">${initial_positions['right_index_mcp_joint']}</param></state_interface><state_interface name="velocity" /></joint>
         <joint name="right_index_pip_joint"><command_interface name="position" /><state_interface name="position"><param name="initial_value">${initial_positions['right_index_pip_joint']}</param></state_interface><state_interface name="velocity" /></joint>
+        <joint name="right_middle_abad_joint"><command_interface name="position" /><state_interface name="position"><param name="initial_value">${initial_positions['right_middle_abad_joint']}</param></state_interface><state_interface name="velocity" /></joint>
+        <joint name="right_middle_mcp_joint"><command_interface name="position" /><state_interface name="position"><param name="initial_value">${initial_positions['right_middle_mcp_joint']}</param></state_interface><state_interface name="velocity" /></joint>
         <joint name="right_middle_pip_joint"><command_interface name="position" /><state_interface name="position"><param name="initial_value">${initial_positions['right_middle_pip_joint']}</param></state_interface><state_interface name="velocity" /></joint>
-        <joint name="right_ring_abad_joint"><command_interface name="position" /><state_interface name="position"><param name="initial_value">${initial_positions['right_ring_abad_joint']}</param></state_interface><state_interface name="velocity" /></joint>
-        <joint name="right_ring_pip_joint"><command_interface name="position" /><state_interface name="position"><param name="initial_value">${initial_positions['right_ring_pip_joint']}</param></state_interface><state_interface name="velocity" /></joint>
-        <joint name="right_pinky_abad_joint"><command_interface name="position" /><state_interface name="position"><param name="initial_value">${initial_positions['right_pinky_abad_joint']}</param></state_interface><state_interface name="velocity" /></joint>
-        <joint name="right_pinky_pip_joint"><command_interface name="position" /><state_interface name="position"><param name="initial_value">${initial_positions['right_pinky_pip_joint']}</param></state_interface><state_interface name="velocity" /></joint>
+        <joint name="right_ring_mcp_joint"><command_interface name="position" /><state_interface name="position"><param name="initial_value">${initial_positions['right_ring_mcp_joint']}</param></state_interface><state_interface name="velocity" /></joint>
+        <joint name="right_pinky_mcp_joint"><command_interface name="position" /><state_interface name="position"><param name="initial_value">${initial_positions['right_pinky_mcp_joint']}</param></state_interface><state_interface name="velocity" /></joint>
       </xacro:if>
     </ros2_control>

File: src/agx_arm_moveit/config/agx_arm.srdf.xacro (robot description, xacro)
@@ -83,11 +83,13 @@
       <joint name="${side}_thumb_abad_joint" />
       <joint name="${side}_thumb_mcp_joint" />
+      <joint name="${side}_thumb_pip_joint" />
       <joint name="${side}_index_abad_joint" />
+      <joint name="${side}_index_mcp_joint" />
       <joint name="${side}_index_pip_joint" />
+      <joint name="${side}_middle_abad_joint" />
+      <joint name="${side}_middle_mcp_joint" />
       <joint name="${side}_middle_pip_joint" />
-      <joint name="${side}_ring_abad_joint" />
-      <joint name="${side}_ring_pip_joint" />
-      <joint name="${side}_pinky_abad_joint" />
-      <joint name="${side}_pinky_pip_joint" />
+      <joint name="${side}_ring_mcp_joint" />
+      <joint name="${side}_pinky_mcp_joint" />
     </group>
     <end_effector name="${side}_omnihand_eef" parent_link="${end_effector_parent_link}" group="hand" parent_group="${planning_group_name}" />
@@ -96,41 +98,48 @@
       <joint name="${side}_thumb_abad_joint" value="0.0" />
       <joint name="${side}_thumb_mcp_joint" value="0.0" />
+      <joint name="${side}_thumb_pip_joint" value="0.0" />
       <joint name="${side}_index_abad_joint" value="0.0" />
+      <joint name="${side}_index_mcp_joint" value="0.0" />
       <joint name="${side}_index_pip_joint" value="0.0" />
+      <joint name="${side}_middle_abad_joint" value="0.0" />
+      <joint name="${side}_middle_mcp_joint" value="0.0" />
       <joint name="${side}_middle_pip_joint" value="0.0" />
-      <joint name="${side}_ring_abad_joint" value="0.0" />
-      <joint name="${side}_ring_pip_joint" value="0.0" />
-      <joint name="${side}_pinky_abad_joint" value="0.0" />
-      <joint name="${side}_pinky_pip_joint" value="0.0" />
+      <joint name="${side}_ring_mcp_joint" value="0.0" />
+      <joint name="${side}_pinky_mcp_joint" value="0.0" />
     </group_state>
     <group_state name="hand_half_close" group="hand">
-      <joint name="${side}_thumb_roll_joint" value="${-0.25 if side == 'left' else 0.25}" />
-      <joint name="${side}_thumb_abad_joint" value="${0.6 if side == 'left' else -0.6}" />
-      <joint name="${side}_thumb_mcp_joint" value="${-0.35 if side == 'left' else 0.35}" />
-      <joint name="${side}_index_abad_joint" value="${0.05 if side == 'left' else -0.05}" />
-      <joint name="${side}_index_pip_joint" value="0.7" />
-      <joint name="${side}_middle_pip_joint" value="0.7" />
-      <joint name="${side}_ring_abad_joint" value="${-0.05 if side == 'left' else 0.05}" />
-      <joint name="${side}_ring_pip_joint" value="0.7" />
-      <joint name="${side}_pinky_abad_joint" value="${-0.05 if side == 'left' else 0.05}" />
-      <joint name="${side}_pinky_pip_joint" value="0.7" />
+      <joint name="${side}_thumb_roll_joint" value="${-0.2 if side == 'left' else 0.2}" />
+      <joint name="${side}_thumb_abad_joint" value="${0.3 if side == 'left' else -0.3}" />
+      <joint name="${side}_thumb_mcp_joint" value="-0.25" />
+      <joint name="${side}_thumb_pip_joint" value="-0.3" />
+      <joint name="${side}_index_abad_joint" value="0.0" />
+      <joint name="${side}_index_mcp_joint" value="0.6" />
+      <joint name="${side}_index_pip_joint" value="0.6" />
+      <joint name="${side}_middle_abad_joint" value="0.0" />
+      <joint name="${side}_middle_mcp_joint" value="0.6" />
+      <joint name="${side}_middle_pip_joint" value="0.6" />
+      <joint name="${side}_ring_mcp_joint" value="0.6" />
+      <joint name="${side}_pinky_mcp_joint" value="0.6" />
     </group_state>
     <group_state name="hand_close" group="hand">
-      <joint name="${side}_thumb_roll_joint" value="${-0.45 if side == 'left' else 0.45}" />
-      <joint name="${side}_thumb_abad_joint" value="${1.0 if side == 'left' else -1.0}" />
-      <joint name="${side}_thumb_mcp_joint" value="${-0.6 if side == 'left' else 0.6}" />
-      <joint name="${side}_index_abad_joint" value="${0.1 if side == 'left' else -0.1}" />
-      <joint name="${side}_index_pip_joint" value="1.2" />
-      <joint name="${side}_middle_pip_joint" value="1.2" />
-      <joint name="${side}_ring_abad_joint" value="${-0.1 if side == 'left' else 0.1}" />
-      <joint name="${side}_ring_pip_joint" value="1.2" />
-      <joint name="${side}_pinky_abad_joint" value="${-0.1 if side == 'left' else 0.1}" />
-      <joint name="${side}_pinky_pip_joint" value="1.2" />
-    </group_state>
-    <passive_joint name="${side}_thumb_pip_joint" />
+      <joint name="${side}_thumb_roll_joint" value="${-0.4 if side == 'left' else 0.4}" />
+      <joint name="${side}_thumb_abad_joint" value="${0.5 if side == 'left' else -0.5}" />
+      <joint name="${side}_thumb_mcp_joint" value="-0.5" />
+      <joint name="${side}_thumb_pip_joint" value="-0.6" />
+      <joint name="${side}_index_abad_joint" value="0.0" />
+      <joint name="${side}_index_mcp_joint" value="1.1" />
+      <joint name="${side}_index_pip_joint" value="1.1" />
+      <joint name="${side}_middle_abad_joint" value="0.0" />
+      <joint name="${side}_middle_mcp_joint" value="1.1" />
+      <joint name="${side}_middle_pip_joint" value="1.1" />
+      <joint name="${side}_ring_mcp_joint" value="1.2" />
+      <joint name="${side}_pinky_mcp_joint" value="1.2" />
+    </group_state>
     <passive_joint name="${side}_thumb_dip_joint" />
     <passive_joint name="${side}_index_dip_joint" />
     <passive_joint name="${side}_middle_dip_joint" />
+    <passive_joint name="${side}_ring_pip_joint" />
     <passive_joint name="${side}_ring_dip_joint" />
+    <passive_joint name="${side}_pinky_pip_joint" />
     <passive_joint name="${side}_pinky_dip_joint" />
     <disable_collisions link1="${arm_link_prefix}link7" link2="${arm_link_prefix}omnihand_flange" reason="Adjacent" />
@@ -139,21 +148,24 @@
     <disable_collisions link1="${arm_link_prefix}omnihand_flange" link2="${side}_palm" reason="Adjacent" />
     <disable_collisions link1="${side}_base_link" link2="${side}_palm" reason="Adjacent" />
-    <disable_collisions link1="${side}_palm" link2="${side}_thumb_roll" reason="Adjacent" />
-    <disable_collisions link1="${side}_palm" link2="${side}_index_abad" reason="Adjacent" />
-    <disable_collisions link1="${side}_palm" link2="${side}_middle_abad" reason="Adjacent" />
-    <disable_collisions link1="${side}_palm" link2="${side}_ring_abad" reason="Adjacent" />
-    <disable_collisions link1="${side}_palm" link2="${side}_pinky_abad" reason="Adjacent" />
-    <disable_collisions link1="${side}_thumb_roll" link2="${side}_thumb_abad" reason="Adjacent" />
-    <disable_collisions link1="${side}_thumb_abad" link2="${side}_thumb_mcp" reason="Adjacent" />
-    <disable_collisions link1="${side}_thumb_mcp" link2="${side}_thumb_pip" reason="Adjacent" />
-    <disable_collisions link1="${side}_thumb_pip" link2="${side}_thumb_dip" reason="Adjacent" />
-    <disable_collisions link1="${side}_index_abad" link2="${side}_index_pip" reason="Adjacent" />
-    <disable_collisions link1="${side}_index_pip" link2="${side}_index_dip" reason="Adjacent" />
-    <disable_collisions link1="${side}_middle_abad" link2="${side}_middle_pip" reason="Adjacent" />
-    <disable_collisions link1="${side}_middle_pip" link2="${side}_middle_dip" reason="Adjacent" />
-    <disable_collisions link1="${side}_ring_abad" link2="${side}_ring_pip" reason="Adjacent" />
-    <disable_collisions link1="${side}_ring_pip" link2="${side}_ring_dip" reason="Adjacent" />
-    <disable_collisions link1="${side}_pinky_abad" link2="${side}_pinky_pip" reason="Adjacent" />
-    <disable_collisions link1="${side}_pinky_pip" link2="${side}_pinky_dip" reason="Adjacent" />
+    <disable_collisions link1="${side}_palm" link2="${side}_thumb_roll_link" reason="Adjacent" />
+    <disable_collisions link1="${side}_palm" link2="${side}_thumb_abad_link" reason="Never" />
+    <disable_collisions link1="${side}_palm" link2="${side}_index_abad_link" reason="Adjacent" />
+    <disable_collisions link1="${side}_palm" link2="${side}_middle_abad_link" reason="Adjacent" />
+    <disable_collisions link1="${side}_palm" link2="${side}_ring_mcp_link" reason="Adjacent" />
+    <disable_collisions link1="${side}_palm" link2="${side}_pinky_mcp_link" reason="Adjacent" />
+    <disable_collisions link1="${side}_thumb_roll_link" link2="${side}_thumb_abad_link" reason="Adjacent" />
+    <disable_collisions link1="${side}_thumb_abad_link" link2="${side}_thumb_mcp_link" reason="Adjacent" />
+    <disable_collisions link1="${side}_thumb_mcp_link" link2="${side}_thumb_pip_link" reason="Adjacent" />
+    <disable_collisions link1="${side}_thumb_pip_link" link2="${side}_thumb_dip_link" reason="Adjacent" />
+    <disable_collisions link1="${side}_index_abad_link" link2="${side}_index_mcp_link" reason="Adjacent" />
+    <disable_collisions link1="${side}_index_mcp_link" link2="${side}_index_pip_link" reason="Adjacent" />
+    <disable_collisions link1="${side}_index_pip_link" link2="${side}_index_dip_link" reason="Adjacent" />
+    <disable_collisions link1="${side}_middle_abad_link" link2="${side}_middle_mcp_link" reason="Adjacent" />
+    <disable_collisions link1="${side}_middle_mcp_link" link2="${side}_middle_pip_link" reason="Adjacent" />
+    <disable_collisions link1="${side}_middle_pip_link" link2="${side}_middle_dip_link" reason="Adjacent" />
+    <disable_collisions link1="${side}_ring_mcp_link" link2="${side}_ring_pip_link" reason="Adjacent" />
+    <disable_collisions link1="${side}_ring_pip_link" link2="${side}_ring_dip_link" reason="Adjacent" />
+    <disable_collisions link1="${side}_pinky_mcp_link" link2="${side}_pinky_pip_link" reason="Adjacent" />
+    <disable_collisions link1="${side}_pinky_pip_link" link2="${side}_pinky_dip_link" reason="Adjacent" />
   </xacro:macro>
   <!-- ======================== ARM GROUPS ======================== -->

File: src/agx_arm_sim/agx_arm_description/agx_arm_urdf/omnihand/urdf/omnihand_left_hand.xacro (robot description, xacro)
@@ -1,5 +1,5 @@
 <?xml version="1.0"?>
 <robot xmlns:xacro="http://www.ros.org/wiki/xacro" name="omnihand">
-  <xacro:include filename="$(find agx_arm_description)/agx_arm_urdf/omnihand/urdf/xacro/hand.xacro" />
+  <xacro:include filename="$(find agx_arm_description)/agx_arm_urdf/omnihand/urdf/xacro_pro/hand.xacro" />
   <link name="left_base_link">
     <visual>

File: src/agx_arm_sim/agx_arm_description/agx_arm_urdf/omnihand/urdf/omnihand_right_hand.xacro (robot description, xacro)
@@ -1,5 +1,5 @@
 <?xml version="1.0"?>
 <robot xmlns:xacro="http://www.ros.org/wiki/xacro" name="omnihand">
-  <xacro:include filename="$(find agx_arm_description)/agx_arm_urdf/omnihand/urdf/xacro/hand.xacro" />
+  <xacro:include filename="$(find agx_arm_description)/agx_arm_urdf/omnihand/urdf/xacro_pro/hand.xacro" />
   <link name="right_base_link">
     <visual>

File: src/duo_body_description/urdf/nero_arm_macro.xacro (robot description, xacro)
@@ -1,5 +1,5 @@
 <?xml version="1.0"?>
 <robot xmlns:xacro="http://www.ros.org/wiki/xacro">
-  <xacro:include filename="$(find agx_arm_description)/agx_arm_urdf/omnihand/urdf/xacro/hand.xacro"/>
+  <xacro:include filename="$(find agx_arm_description)/agx_arm_urdf/omnihand/urdf/xacro_pro/hand.xacro"/>
   <xacro:macro name="nero_arm" params="prefix">
     <link name="${prefix}base_link">
